Commit message: 全驱动+机械臂

File: src/dragonfly_arm/urdf/dragonfly_arm.urdf.xacro (robot description, xacro)
@@ -2,205 +2,31 @@
 <robot xmlns:xacro="http://www.ros.org/wiki/xacro" name="dragonfly_arm">
   <xacro:arg name="use_sim_time" default="true"/>
-  <material name="dragonfly_blue">
-    <color rgba="0.10 0.38 0.78 1.0"/>
-  </material>
-  <material name="dragonfly_dark">
-    <color rgba="0.10 0.12 0.16 1.0"/>
-  </material>
-  <material name="dragonfly_orange">
-    <color rgba="0.95 0.36 0.08 1.0"/>
-  </material>
-  <material name="dragonfly_silver">
-    <color rgba="0.62 0.66 0.72 1.0"/>
-  </material>
-  <xacro:macro name="box_inertial" params="mass x y z origin_xyz">
-    <inertial>
-      <origin xyz="${origin_xyz}" rpy="0 0 0"/>
-      <mass value="${mass}"/>
-      <inertia
-        ixx="${mass * (y * y + z * z) / 12.0}" ixy="0" ixz="0"
-        iyy="${mass * (x * x + z * z) / 12.0}" iyz="0"
-        izz="${mass * (x * x + y * y) / 12.0}"/>
-    </inertial>
-  </xacro:macro>
-  <xacro:macro name="cylinder_inertial" params="mass radius length origin_xyz">
-    <inertial>
-      <origin xyz="${origin_xyz}" rpy="0 0 0"/>
-      <mass value="${mass}"/>
-      <inertia
-        ixx="${mass * (3.0 * radius * radius + length * length) / 12.0}" ixy="0" ixz="0"
-        iyy="${mass * (3.0 * radius * radius + length * length) / 12.0}" iyz="0"
-        izz="${mass * radius * radius / 2.0}"/>
-    </inertial>
-  </xacro:macro>
+  <xacro:property name="cfg" value="${xacro.load_yaml('../config/model_dimensions.yaml')}"/>
+  <xacro:property name="meas" value="${cfg.measured}"/>
+  <xacro:property name="est" value="${cfg.estimated}"/>
+  <xacro:property name="sim" value="${cfg.simulation}"/>
+  <xacro:include filename="geometry_macros.xacro"/>
+  <xacro:include filename="vector_platform.xacro"/>
+  <xacro:include filename="five_axis_arm.xacro"/>
+  <!-- Fixed-base kinematic demonstrator; this constraint must be removed
+       together with adding flight physics, NOT simply when adding wind. -->
   <link name="world"/>
-  <gazebo reference="world">
-    <static>true</static>
-  </gazebo>
-  <joint name="world_to_base" type="fixed">
-    <parent link="world"/>
-    <child link="base_link"/>
-    <origin xyz="0 0 0" rpy="0 0 0"/>
-  </joint>
-  <link name="base_link">
-    <visual>
-      <origin xyz="0 0 0.06" rpy="0 0 0"/>
-      <geometry><cylinder radius="0.16" length="0.12"/></geometry>
-      <material name="dragonfly_dark"/>
-    </visual>
-    <collision>
-      <origin xyz="0 0 0.06" rpy="0 0 0"/>
-      <geometry><cylinder radius="0.16" length="0.12"/></geometry>
-    </collision>
-    <xacro:cylinder_inertial mass="12.0" radius="0.16" length="0.12" origin_xyz="0 0 0.06"/>
-  </link>
-  <joint name="joint_1" type="revolute">
-    <parent link="base_link"/>
-    <child link="shoulder_link"/>
-    <origin xyz="0 0 0.12" rpy="0 0 0"/>
-    <axis xyz="0 0 1"/>
-    <limit lower="-${pi}" upper="${pi}" effort="120" velocity="1.2"/>
-    <dynamics damping="0.60" friction="0.05"/>
-  </joint>
-  <link name="shoulder_link">
-    <visual>
-      <origin xyz="0 0 0.09" rpy="0 0 0"/>
-      <geometry><cylinder radius="0.10" length="0.18"/></geometry>
-      <material name="dragonfly_blue"/>
-    </visual>
-    <collision>
-      <origin xyz="0 0 0.09" rpy="0 0 0"/>
-      <geometry><cylinder radius="0.10" length="0.18"/></geometry>
-    </collision>
-    <xacro:cylinder_inertial mass="8.0" radius="0.10" length="0.18" origin_xyz="0 0 0.09"/>
-  </link>
-  <joint name="joint_2" type="revolute">
-    <parent link="shoulder_link"/>
-    <child link="upper_arm_link"/>
-    <origin xyz="0 0 0.18" rpy="0 0 0"/>
-    <axis xyz="0 1 0"/>
-    <limit lower="-2.30" upper="2.30" effort="100" velocity="1.2"/>
-    <dynamics damping="0.80" friction="0.05"/>
-  </joint>
-  <link name="upper_arm_link">
-    <visual>
-      <origin xyz="0 0 0.17" rpy="0 0 0"/>
-      <geometry><box size="0.11 0.13 0.34"/></geometry>
-      <material name="dragonfly_orange"/>
-    </visual>
-    <collision>
-      <origin xyz="0 0 0.17" rpy="0 0 0"/>
-      <geometry><box size="0.11 0.13 0.34"/></geometry>
-    </collision>
-    <xacro:box_inertial mass="6.0" x="0.11" y="0.13" z="0.34" origin_xyz="0 0 0.17"/>
-  </link>
-  <joint name="joint_3" type="revolute">
-    <parent link="upper_arm_link"/>
-    <child link="forearm_link"/>
-    <origin xyz="0 0 0.34" rpy="0 0 0"/>
-    <axis xyz="0 1 0"/>
-    <limit lower="-2.50" upper="2.50" effort="80" velocity="1.3"/>
-    <dynamics damping="0.65" friction="0.04"/>
-  </joint>
-  <link name="forearm_link">
-    <visual>
-      <origin xyz="0 0 0.15" rpy="0 0 0"/>
-      <geometry><box size="0.09 0.11 0.30"/></geometry>
-      <material name="dragonfly_blue"/>
-    </visual>
-    <collision>
-      <origin xyz="0 0 0.15" rpy="0 0 0"/>
-      <geometry><box size="0.09 0.11 0.30"/></geometry>
-    </collision>
-    <xacro:box_inertial mass="4.0" x="0.09" y="0.11" z="0.30" origin_xyz="0 0 0.15"/>
-  </link>
-  <joint name="joint_4" type="revolute">
-    <parent link="forearm_link"/>
-    <child link="wrist_1_link"/>
-    <origin xyz="0 0 0.30" rpy="0 0 0"/>
-    <axis xyz="1 0 0"/>
-    <limit lower="-${pi}" upper="${pi}" effort="40" velocity="1.8"/>
-    <dynamics damping="0.35" friction="0.03"/>
-  </joint>
-  <link name="wrist_1_link">
-    <visual>
-      <origin xyz="0 0 0.07" rpy="0 0 0"/>
-      <geometry><cylinder radius="0.07" length="0.14"/></geometry>
-      <material name="dragonfly_silver"/>
-    </visual>
-    <collision>
-      <origin xyz="0 0 0.07" rpy="0 0 0"/>
-      <geometry><cylinder radius="0.07" length="0.14"/></geometry>
-    </collision>
-    <xacro:cylinder_inertial mass="2.0" radius="0.07" length="0.14" origin_xyz="0 0 0.07"/>
-  </link>
-  <joint name="joint_5" type="revolute">
-    <parent link="wrist_1_link"/>
-    <child link="wrist_2_link"/>
-    <origin xyz="0 0 0.14" rpy="0 0 0"/>
-    <axis xyz="0 1 0"/>
-    <limit lower="-2.10" upper="2.10" effort="30" velocity="1.8"/>
-    <dynamics damping="0.30" friction="0.02"/>
-  </joint>
-  <link name="wrist_2_link">
-    <visual>
-      <origin xyz="0 0 0.06" rpy="0 0 0"/>
-      <geometry><cylinder radius="0.06" length="0.12"/></geometry>
-      <material name="dragonfly_orange"/>
-    </visual>
-    <collision>
-      <origin xyz="0 0 0.06" rpy="0 0 0"/>
-      <geometry><cylinder radius="0.06" length="0.12"/></geometry>
-    </collision>
-    <xacro:cylinder_inertial mass="1.2" radius="0.06" length="0.12" origin_xyz="0 0 0.06"/>
-  </link>
-  <joint name="joint_6" type="revolute">
-    <parent link="wrist_2_link"/>
-    <child link="tool0"/>
-    <origin xyz="0 0 0.12" rpy="0 0 0"/>
-    <axis xyz="1 0 0"/>
-    <limit lower="-${pi}" upper="${pi}" effort="20" velocity="2.0"/>
-    <dynamics damping="0.25" friction="0.02"/>
-  </joint>
-  <link name="tool0">
-    <visual>
-      <origin xyz="0 0 0.06" rpy="0 0 0"/>
-      <geometry><box size="0.06 0.10 0.12"/></geometry>
-      <material name="dragonfly_dark"/>
-    </visual>
-    <collision>
-      <origin xyz="0 0 0.06" rpy="0 0 0"/>
-      <geometry><box size="0.06 0.10 0.12"/></geometry>
-    </collision>
-    <xacro:box_inertial mass="0.8" x="0.06" y="0.10" z="0.12" origin_xyz="0 0 0.06"/>
-  </link>
+  <gazebo reference="world"><static>true</static></gazebo>
+  <xacro:vector_platform/>
+  <xacro:five_axis_arm/>
   <ros2_control name="GazeboSystem" type="system">
-    <hardware>
-      <plugin>gazebo_ros2_control/GazeboSystem</plugin>
-    </hardware>
-    <xacro:macro name="controlled_joint" params="name lower upper">
-      <joint name="${name}">
-        <command_interface name="position">
-          <param name="min">${lower}</param>
-          <param name="max">${upper}</param>
-        </command_interface>
-        <state_interface name="position"/>
-        <state_interface name="velocity"/>
-      </joint>
-    </xacro:macro>
-    <xacro:controlled_joint name="joint_1" lower="-${pi}" upper="${pi}"/>
-    <xacro:controlled_joint name="joint_2" lower="-2.30" upper="2.30"/>
-    <xacro:controlled_joint name="joint_3" lower="-2.50" upper="2.50"/>
-    <xacro:controlled_joint name="joint_4" lower="-${pi}" upper="${pi}"/>
-    <xacro:controlled_joint name="joint_5" lower="-2.10" upper="2.10"/>
-    <xacro:controlled_joint name="joint_6" lower="-${pi}" upper="${pi}"/>
+    <hardware><plugin>gazebo_ros2_control/GazeboSystem</plugin></hardware>
+    <xacro:controlled_joint name="joint_1"/>
+    <xacro:controlled_joint name="joint_2"/>
+    <xacro:controlled_joint name="joint_3"/>
+    <xacro:controlled_joint name="joint_4"/>
+    <xacro:controlled_joint name="joint_5"/>
+    <xacro:controlled_joint name="unit_a_outer_joint"/>
+    <xacro:controlled_joint name="unit_a_inner_joint"/>
+    <xacro:controlled_joint name="unit_b_outer_joint"/>
+    <xacro:controlled_joint name="unit_b_inner_joint"/>
+    <xacro:controlled_joint name="unit_c_outer_joint"/>
+    <xacro:controlled_joint name="unit_c_inner_joint"/>
   </ros2_control>
-  <gazebo reference="base_link"><material>Gazebo/Black</material></gazebo>
-  <gazebo reference="shoulder_link"><material>Gazebo/Blue</material></gazebo>
-  <gazebo reference="upper_arm_link"><material>Gazebo/Orange</material></gazebo>
-  <gazebo reference="forearm_link"><material>Gazebo/Blue</material></gazebo>
-  <gazebo reference="wrist_1_link"><material>Gazebo/Grey</material></gazebo>
-  <gazebo reference="wrist_2_link"><material>Gazebo/Orange</material></gazebo>
-  <gazebo reference="tool0"><material>Gazebo/Black</material></gazebo>
   <gazebo>
     <plugin name="gazebo_ros2_control" filename="libgazebo_ros2_control.so">

Commit message: 完善原生 PX4 双臂仿真并更新工程进度

File: src/dragonfly_arm/urdf/dragonfly_arm.urdf.xacro (robot description, xacro)
@@ -5,4 +5,7 @@
   <xacro:property name="meas" value="${cfg.measured}"/>
   <xacro:property name="kin" value="${cfg.arm_kinematics}"/>
+  <xacro:property name="hardware" value="${cfg.arm_hardware}"/>
+  <xacro:property name="weights" value="${cfg.arm_dynamics.mass_weights}"/>
+  <xacro:property name="mass_scale" value="${meas.arm_mass/(weights.base+weights.column+weights.upper_arm+weights.forearm+weights.wrist+weights.gripper)}"/>
   <xacro:property name="est" value="${cfg.estimated}"/>
   <xacro:property name="sim" value="${cfg.simulation}"/>

File: src/dragonfly_arm/urdf/five_axis_arm.xacro (robot description, xacro)
@@ -2,25 +2,35 @@
 <robot xmlns:xacro="http://www.ros.org/wiki/xacro">
   <!-- RoArm-M3 joint angles use the firmware convention directly. -->
-  <xacro:macro name="arm_joint" params="name parent child xyz axis lower upper rpy:='0 0 0'">
+  <xacro:macro name="arm_joint" params="name parent child xyz axis lower upper actuator rpy:='0 0 0'">
+    <xacro:property name="drive" value="${hardware.joints[actuator]}"/>
+    <xacro:property name="peak_effort" value="${hardware.servos[drive.servo].stall_torque_kgf_cm*hardware.kgf_cm_to_nm*drive.count}"/>
     <joint name="${name}" type="revolute">
       <parent link="${parent}"/><child link="${child}"/>
       <origin xyz="${xyz}" rpy="${rpy}"/>
       <axis xyz="${axis}"/>
-      <limit lower="${lower}" upper="${upper}" effort="${sim.arm_effort}" velocity="${sim.arm_velocity}"/>
+      <limit lower="${lower}" upper="${upper}" effort="${peak_effort}" velocity="${sim.arm_velocity}"/>
       <dynamics damping="0.1" friction="0.01"/>
     </joint>
   </xacro:macro>
+  <!-- Exact manufacturer casing size; placement / bracket outlines are estimates. -->
+  <xacro:macro name="arm_servo_shape" params="xyz model:=ST3215">
+    <xacro:property name="servo" value="${hardware.servos[model]}"/>
+    <xacro:box_shape x="${servo.body_height}" y="${servo.body_width}" z="${servo.body_length}"
+      xyz="${xyz}" material="servo"/>
+  </xacro:macro>
   <!-- A paired-rail moving link from its joint origin to (dx, 0, dz). -->
-  <xacro:macro name="arm_segment" params="name dx dz mass">
+  <xacro:macro name="arm_segment" params="name dx dz mass outer_width servo:=true">
     <xacro:property name="length" value="${sqrt(dx*dx+dz*dz)}"/>
     <xacro:property name="pitch" value="${atan2(dx,dz)}"/>
     <link name="${name}">
       <xacro:box_shape x="${est.arm_rail_depth}" y="${est.arm_rail_width}" z="${length-0.012}"
-        xyz="${dx/2} ${est.arm_half_width} ${dz/2}" rpy="0 ${pitch} 0"/>
+        xyz="${dx/2} ${(outer_width-est.arm_rail_width)/2} ${dz/2}" rpy="0 ${pitch} 0"/>
       <xacro:box_shape x="${est.arm_rail_depth}" y="${est.arm_rail_width}" z="${length-0.012}"
-        xyz="${dx/2} ${-est.arm_half_width} ${dz/2}" rpy="0 ${pitch} 0"/>
-      <xacro:box_shape x="0.026" y="0.050" z="0.030" xyz="0 0 0.015" material="servo"/>
+        xyz="${dx/2} ${-(outer_width-est.arm_rail_width)/2} ${dz/2}" rpy="0 ${pitch} 0"/>
+      <xacro:if value="${servo}">
+        <xacro:arm_servo_shape xyz="0 0 ${hardware.servos.ST3215.body_length/2}"/>
+      </xacro:if>
       <xacro:cylinder_shape radius="0.008" length="0.058" rpy="${pi/2} 0 0" material="metal"/>
-      <xacro:box_inertial mass="${mass}" x="0.030" y="${2*est.arm_half_width+est.arm_rail_width}" z="${length}"
+      <xacro:box_inertial mass="${mass}" x="${hardware.servos.ST3215.body_height}" y="${outer_width}" z="${length}"
         xyz="${dx/2} 0 ${dz/2}" rpy="0 ${pitch} 0"/>
     </link>
@@ -40,41 +50,54 @@
     </joint>
     <link name="${prefix}_base_link">
-      <xacro:box_shape x="0.070" y="0.065" z="0.008" xyz="0 0 0.004"/>
-      <xacro:cylinder_shape radius="0.025" length="0.030" xyz="0 0 0.019" material="servo"/>
-      <xacro:box_inertial mass="${sim.arm_base_mass}" x="0.070" y="0.065" z="0.038" xyz="0 0 0.019"/>
+      <xacro:box_shape x="0.070" y="0.065" z="${meas.arm_base_plate_thickness}" xyz="0 0 ${meas.arm_base_plate_thickness/2}"/>
+      <xacro:box_shape x="${hardware.servos.ST3215.body_length}" y="${hardware.servos.ST3215.body_width}"
+        z="${hardware.servos.ST3215.body_height}" xyz="0 0 ${meas.arm_base_plate_thickness+hardware.servos.ST3215.body_height/2}" material="servo"/>
+      <xacro:box_inertial mass="${mass_scale*weights.base}" x="0.070" y="0.065"
+        z="${meas.arm_base_plate_thickness+hardware.servos.ST3215.body_height}"
+        xyz="0 0 ${(meas.arm_base_plate_thickness+hardware.servos.ST3215.body_height)/2}"/>
     </link>
     <xacro:arm_joint name="${prefix}_joint_1" parent="${prefix}_base_link" child="${prefix}_column_link"
       xyz="0 0 0" axis="0 0 1"
-      lower="${kin.joint_limits.base.lower}" upper="${kin.joint_limits.base.upper}"/>
+      lower="${kin.joint_limits.base.lower}" upper="${kin.joint_limits.base.upper}" actuator="base"/>
     <link name="${prefix}_column_link">
-      <xacro:box_shape x="0.045" y="0.055" z="${kin.base_to_shoulder}"
-        xyz="0 0 ${kin.base_to_shoulder/2}" material="servo"/>
-      <xacro:box_shape x="0.070" y="0.060" z="0.010"
-        xyz="0 0 ${kin.base_to_shoulder-0.005}"/>
-      <xacro:box_inertial mass="${sim.shoulder_mass}" x="0.055" y="0.060" z="${kin.base_to_shoulder}"
+      <xacro:property name="bracket_bottom" value="${kin.base_to_shoulder-meas.shoulder_bracket_height}"/>
+      <xacro:property name="shoulder_servo_y" value="${(meas.upper_arm_outer_width+hardware.servos.ST3215.body_width)/2}"/>
+      <xacro:box_shape x="0.045" y="0.055" z="${bracket_bottom}"
+        xyz="0 0 ${bracket_bottom/2}" material="servo"/>
+      <xacro:box_shape x="0.050" y="0.003" z="${meas.shoulder_bracket_height}"
+        xyz="0 ${shoulder_servo_y+hardware.servos.ST3215.body_width/2+0.0015} ${bracket_bottom+meas.shoulder_bracket_height/2}"/>
+      <xacro:box_shape x="0.050" y="0.003" z="${meas.shoulder_bracket_height}"
+        xyz="0 ${-shoulder_servo_y-hardware.servos.ST3215.body_width/2-0.0015} ${bracket_bottom+meas.shoulder_bracket_height/2}"/>
+      <xacro:arm_servo_shape xyz="0 ${shoulder_servo_y} ${kin.base_to_shoulder-hardware.servos.ST3215.body_length/2}"/>
+      <xacro:arm_servo_shape xyz="0 ${-shoulder_servo_y} ${kin.base_to_shoulder-hardware.servos.ST3215.body_length/2}"/>
+      <xacro:box_inertial mass="${mass_scale*weights.column}" x="0.055"
+        y="${2*shoulder_servo_y+hardware.servos.ST3215.body_width+0.006}" z="${kin.base_to_shoulder}"
         xyz="0 0 ${kin.base_to_shoulder/2}"/>
     </link>
     <xacro:arm_joint name="${prefix}_joint_2" parent="${prefix}_column_link" child="${prefix}_upper_arm_link"
       xyz="0 0 ${kin.base_to_shoulder}" axis="0 1 0"
-      lower="${kin.joint_limits.shoulder.lower}" upper="${kin.joint_limits.shoulder.upper}"/>
+      lower="${kin.joint_limits.shoulder.lower}" upper="${kin.joint_limits.shoulder.upper}" actuator="shoulder"/>
     <xacro:arm_segment name="${prefix}_upper_arm_link"
-      dx="${kin.shoulder_to_elbow_x}" dz="${kin.shoulder_to_elbow_z}" mass="${sim.upper_arm_mass}"/>
+      dx="${kin.shoulder_to_elbow_x}" dz="${kin.shoulder_to_elbow_z}" mass="${mass_scale*weights.upper_arm}"
+      outer_width="${meas.upper_arm_outer_width}" servo="false"/>
     <xacro:arm_joint name="${prefix}_joint_3" parent="${prefix}_upper_arm_link" child="${prefix}_forearm_link"
       xyz="${kin.shoulder_to_elbow_x} 0 ${kin.shoulder_to_elbow_z}" axis="0 1 0"
-      lower="${kin.joint_limits.elbow.lower}" upper="${kin.joint_limits.elbow.upper}"/>
+      lower="${kin.joint_limits.elbow.lower}" upper="${kin.joint_limits.elbow.upper}" actuator="elbow"/>
     <xacro:arm_segment name="${prefix}_forearm_link"
-      dx="${kin.elbow_to_wrist_x}" dz="${kin.elbow_to_wrist_z}" mass="${sim.forearm_mass}"/>
+      dx="${kin.elbow_to_wrist_x}" dz="${kin.elbow_to_wrist_z}" mass="${mass_scale*weights.forearm}"
+      outer_width="${2*est.arm_half_width+est.arm_rail_width}"/>
     <xacro:arm_joint name="${prefix}_joint_4" parent="${prefix}_forearm_link" child="${prefix}_wrist_link"
       xyz="${kin.elbow_to_wrist_x} 0 ${kin.elbow_to_wrist_z}" axis="0 1 0"
-      lower="${kin.joint_limits.wrist.lower}" upper="${kin.joint_limits.wrist.upper}"/>
+      lower="${kin.joint_limits.wrist.lower}" upper="${kin.joint_limits.wrist.upper}" actuator="wrist"/>
     <link name="${prefix}_wrist_link">
-      <xacro:box_shape x="0.040" y="0.052" z="0.035" xyz="0 0 0.0175" material="servo"/>
+      <xacro:arm_servo_shape xyz="0 0 ${hardware.servos.ST3215.body_length/2}"/>
       <xacro:cylinder_shape radius="0.009" length="0.060" rpy="${pi/2} 0 0" material="metal"/>
-      <xacro:box_inertial mass="${sim.wrist_mass}" x="0.040" y="0.052" z="0.035" xyz="0 0 0.0175"/>
+      <xacro:box_inertial mass="${mass_scale*weights.wrist}" x="${hardware.servos.ST3215.body_height}"
+        y="0.060" z="${hardware.servos.ST3215.body_length}" xyz="0 0 ${hardware.servos.ST3215.body_length/2}"/>
     </link>
     <!-- The roll axis is aligned with the actual offset terminal segment. -->
     <xacro:arm_joint name="${prefix}_joint_5" parent="${prefix}_wrist_link" child="${prefix}_gripper_link"
       xyz="0 0 0" rpy="0 ${tool_pitch} 0" axis="0 0 1"
-      lower="${kin.joint_limits.roll.lower}" upper="${kin.joint_limits.roll.upper}"/>
+      lower="${kin.joint_limits.roll.lower}" upper="${kin.joint_limits.roll.upper}" actuator="roll"/>
     <link name="${prefix}_gripper_link">
       <xacro:box_shape x="${est.arm_rail_depth}" y="${est.arm_rail_width}" z="${tool_length-0.015}"
@@ -82,9 +105,10 @@
       <xacro:box_shape x="${est.arm_rail_depth}" y="${est.arm_rail_width}" z="${tool_length-0.015}"
         xyz="0 ${-est.arm_half_width} ${tool_length/2}"/>
-      <xacro:box_shape x="0.030" y="0.052" z="0.035" xyz="0 0 0.020" material="servo"/>
+      <xacro:arm_servo_shape xyz="0 0 ${hardware.servos.ST3215.body_length/2}"/>
+      <xacro:arm_servo_shape model="ST3215-HS" xyz="0 0 ${tool_length-0.055-hardware.servos['ST3215-HS'].body_length/2}"/>
       <!-- Closed fingers end at tool0; their actuator is intentionally not a sixth joint. -->
       <xacro:box_shape x="0.010" y="0.009" z="0.055" xyz="0 0.017 ${tool_length-0.0275}" rpy="0.16 0 0"/>
       <xacro:box_shape x="0.010" y="0.009" z="0.055" xyz="0 -0.017 ${tool_length-0.0275}" rpy="-0.16 0 0"/>
-      <xacro:box_inertial mass="${sim.gripper_mass}" x="0.035" y="0.055" z="${tool_length}" xyz="0 0 ${tool_length/2}"/>
+      <xacro:box_inertial mass="${mass_scale*weights.gripper}" x="${hardware.servos.ST3215.body_height}" y="0.055" z="${tool_length}" xyz="0 0 ${tool_length/2}"/>
     </link>
     <joint name="${prefix}_gripper_to_tool0" type="fixed">
